Commit message: 未修改完成

File: src/only_robot_arm/urdf/only_robot_arm.urdf (robot description, URDF)
Before this commit: robot only_robot_arm, 9 links, 8 joints
Links:
- added link pollination_tip_tcp
Joints:
- added joint pollination_tip_tcp_joint: type fixed, parent pollination_tip_link, child pollination_tip_tcp, origin xyz=0 0 -0.033433 rpy=0 0 0, axis 0 0 0

Commit message: 回到初始状态

File: src/only_robot_arm/urdf/only_robot_arm.urdf (robot description, URDF)
Before this commit: robot only_robot_arm, 10 links, 9 joints
Links:
- removed link pollination_tip_tcp
Joints:
- removed joint pollination_tip_tcp_joint
